Commit message: Remove unwanted stuff and keep the urdf files

File: tiago_urdf/tiago_pal_gripper.urdf (robot description, URDF)
Before this commit: robot tiago, 48 links, 47 joints
Links:
- link arm_1_link: geometry collision mesh filename=meshes/arm/arm_1_collision.dae scale=1 1 1; visual mesh filename=meshes/arm/arm_1.stl scale=1 1 1
- link arm_2_link: geometry collision mesh filename=meshes/arm/arm_2_collision.dae scale=1 1 1; visual mesh filename=meshes/arm/arm_2.stl scale=1 1 1
- link arm_3_link: geometry collision mesh filename=meshes/arm/arm_3_collision.dae scale=1 1 1; visual mesh filename=meshes/arm/arm_3.stl scale=1 1 1
- link arm_4_link: geometry collision mesh filename=meshes/arm/arm_4_collision.dae scale=1 1 1; visual mesh filename=meshes/arm/arm_4.stl scale=1 1 1
- link arm_5_link: geometry collision mesh filename=meshes/arm/arm_5_collision-wrist-2017.dae scale=1 1 1; visual mesh filename=meshes/arm/arm_5-wrist-2017.stl scale=1 1 1
- link arm_6_link: geometry collision mesh filename=meshes/arm/arm_6_collision-wrist-2017.dae scale=1 1 1; visual mesh filename=meshes/arm/arm_6-wrist-2017.stl scale=1 1 1
- link base_antenna_left_link: geometry collision cylinder length=0.17 radius=0.005; visual mesh filename=meshes/objects/antenna.stl
- link base_antenna_right_link: geometry collision cylinder length=0.17 radius=0.005; visual mesh filename=meshes/objects/antenna.stl
- link base_cover_link: geometry visual mesh filename=meshes/base/base_ring.stl
- link base_laser_link: geometry visual mesh filename=meshes/sensors/sick_tim551.stl
- link base_link: geometry collision mesh filename=meshes/base/base_collision.stl; visual mesh filename=meshes/base/base.stl
- link base_sonar_01_link: geometry visual mesh filename=meshes/sensors/srf05.stl
- link base_sonar_02_link: geometry visual mesh filename=meshes/sensors/srf05.stl
- link base_sonar_03_link: geometry visual mesh filename=meshes/sensors/srf05.stl
- link caster_back_left_1_link: geometry visual mesh filename=meshes/wheels/caster_1.stl
- link caster_back_left_2_link: geometry collision sphere radius=0.025; visual mesh filename=meshes/wheels/caster_2.stl
- link caster_back_right_1_link: geometry visual mesh filename=meshes/wheels/caster_1.stl
- link caster_back_right_2_link: geometry collision sphere radius=0.025; visual mesh filename=meshes/wheels/caster_2.stl
- link caster_front_left_1_link: geometry visual mesh filename=meshes/wheels/caster_1.stl
- link caster_front_left_2_link: geometry collision sphere radius=0.025; visual mesh filename=meshes/wheels/caster_2.stl
- link caster_front_right_1_link: geometry visual mesh filename=meshes/wheels/caster_1.stl
- link caster_front_right_2_link: geometry collision sphere radius=0.025; visual mesh filename=meshes/wheels/caster_2.stl
- link gripper_left_finger_link: geometry collision box size=0.01 0.05 0.11; visual mesh filename=meshes/gripper/gripper_finger_link.stl
- link gripper_link: geometry collision mesh filename=meshes/gripper/gripper_link_collision.stl; visual mesh filename=meshes/gripper/gripper_link.stl
- link gripper_right_finger_link: geometry collision box size=0.01 0.05 0.11; visual mesh filename=meshes/gripper/gripper_finger_link.stl scale=-1 -1 1
- link head_1_link: geometry collision mesh filename=meshes/head/head_1_collision.dae scale=1 1 1; visual mesh filename=meshes/head/head_1.stl scale=1 1 1
- link head_2_link: geometry collision mesh filename=meshes/head/head_2_collision.dae scale=1 1 1; visual mesh filename=meshes/head/head_2.stl scale=1 1 1
- link torso_fixed_link: geometry collision box size=0.25 0.25 0.1; collision box size=0.4 0.25 0.04
- link torso_lift_link: geometry collision mesh filename=meshes/torso/torso_lift_collision_core.dae scale=1 1 1; collision mesh filename=meshes/torso/torso_lift_collision_neck.dae scale=1 1 1
- link wheel_left_link: geometry collision sphere radius=0.0985; visual mesh filename=meshes/wheels/wheel.stl
- link wheel_right_link: geometry collision sphere radius=0.0985; visual mesh filename=meshes/wheels/wheel.stl
